File: track_sensor_board.kicad_pcb (KiCad board)
At the start: 2 copper layers, 111.8 x 96.5 mm, 30 parts, among them J1 Barrel_Jack, J10 Screw_Terminal_01x02, J11 Screw_Terminal_01x02, J2 10-18-1032, J3 10-18-1032, J4 10-18-1032, J5 10-18-1032, J6 10-18-1032, J7 10-18-1032, J8 10-18-1032, J9 10-18-1032, SW1 SW_DIP_x04, U1 MCP23017_SP, U2 TSR_1-2450

Commit message: chore: save after recovery, looks good
Parts:
- A1: footprint Module:Adafruit_Ethernet_Featherwing -> Adafruit:Adafruit_Ethernet_Featherwing
- J2, J3, J4, J5, J6, J7, J8, J9: footprint Connector_Molex:CONN_10-18-1032_MOL -> Conn_Molex:CONN_10-18-1032_MOL

Commit message: feat: mostly updated v1.1
Parts:
- removed JP1: SolderJumper_3_Bridged12, Jumper:SolderJumper-3_P1.3mm_Bridged2Bar12_RoundedPad1.0x1.5mm
- added F1: Fuse, Fuse:Fuseholder_Blade_Mini_Keystone_3568, F.Cu at (118.0, 100.9)
- moved REF** 2.87 mm to (112.4, 102.8), turned to 90 degrees
- moved U2 1.49 mm to (118.2, 117.5)
Connections:
- A3 pad 19: unconnected-(A3-D5-Pad19) -> Net-(A3-D5)
- A3 pad 20: unconnected-(A3-D6-Pad20) -> Net-(A3-D6)
- J1 pad 1: +12V -> Net-(F1-Pad1)
- RN1 pad 1: Net-(JP1-C) -> +5V
- RN2 pad 1: Net-(JP1-C) -> +5V
- U1 pad 19: unconnected-(U1-INTB-Pad19) -> Net-(A3-D5)
- U1 pad 20: unconnected-(U1-INTA-Pad20) -> Net-(A3-D6)
Routing:
- net Net-(A3-D6): track 0.00 -> 26.9 mm
- net Net-(A3-D5): track 0.00 -> 23.8 mm
- net Net-(JP1-C): track 20.8 -> 0.00 mm, vias 2 -> 0
- net +5V: track 125.6 -> 144.8 mm
- net Net-(F1-Pad1): track 0.00 -> 15.3 mm
- net +12V: track 40.7 -> 44.4 mm
- net Net-(U1-~{RESET}): track 13.8 -> 14.5 mm
- net GND: vias 62 -> 72
Other:
- board text added: "1A"
- board text added: "1B"
- board text added: "2A"
- board text added: "2B"
- board text added: "3A"
- board text added: "3B"
- board text added: "4A"
- board text added: "4B"
- board text added: "5A"
- board text added: "5B"
- board text added: "6A"
- board text added: "6B"
- board text added: "7A"
- board text added: "7B"
- board text added: "8A"
- board text added: "8B"
- board text added: "BEAVER RUN SENSOR BOARD V1.1 OLIVER REW 12-23-23"
- board text added: "BOARD ID ON = 0; OFF = 1"
- board text removed: "1"
- board text removed: "2"
- board text removed: "3"
- board text removed: "4"
- board text removed: "5"
- board text removed: "6"
- board text removed: "7"
- board text removed: "8"
- board text removed: "BEAVER RUN SENSOR BOARD V1.0 OLIVER REW 11-4-2023"
- board text removed: "Board ID and last 4 bits of IP addr ON = 0; OFF = 1"

Commit message: feat: cleaned up a bit
Parts:
- moved F1 10.8 mm to (128.3, 104.3), turned to -90 degrees
- moved A1 2.54 mm to (142.2, 74.9)
- moved A3 2.54 mm to (195.6, 74.9)
- moved REF** 1.45 mm to (113.7, 103.4), turned to 0 degrees
- moved U2 1.35 mm to (118.1, 116.1), turned to 90 degrees
Routing:
- net GND: track 0.00 -> 16.2 mm, vias 72 -> 68
- net +12V: track 44.4 -> 32.9 mm
- net Net-(A3-SDA/D20): track 54.2 -> 47.3 mm
- net Net-(F1-Pad1): track 15.3 -> 22.2 mm
- net Net-(A3-SCL/D21): track 45.9 -> 52.8 mm
- net +5V: track 144.8 -> 140.8 mm
- net Net-(RN1-R2): track 70.7 -> 74.2 mm
- net Net-(RN1-R1): track 73.3 -> 76.8 mm
- net +3.3V: track 133.4 -> 136.1 mm
- net Net-(A1-SCK): track 57.0 -> 59.3 mm
- net Net-(RN1-R4): track 53.0 -> 55.0 mm
- net Net-(RN1-R3): track 55.6 -> 57.6 mm
- net Net-(RN1-R8): track 81.9 -> 79.9 mm
- net Net-(RN1-R7): track 79.3 -> 77.3 mm
- net Net-(RN1-R6): track 59.1 -> 57.1 mm
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